File: pcb/Esp32Sensors.kicad_sch (KiCad schematic)
At the start: 47 parts, among them J8 USB4215-03-A_REVA, U1 ESP32-C3-MINI-1, U10 LM393, U11 LM393, U2 DHT11, U3 DS18B20, U4 AHT20, U5 BMP280, U6 MPU-6050, U7 MAX30102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

Commit message: updated pcb files
Connections:
- net at U1.26 (GPIO18/USB_D-): now also J8.A7 (DN1), J8.B7 (DN2)
- net at U1.27 (GPIO19/USB_D+): now also J8.A6 (DP1), J8.B6 (DP2)
Changed lines of the file:
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@@
+	)
+	(junction
+		(at 226.06 63.5)
+		(diameter 0)
+		(color 0 0 0 0)
 	)
 	(junction
@@
 	)
 	(junction
+		(at 228.6 49.53)
+		(diameter 0)
+		(color 0 0 0 0)
+	)
+	(junction
 		(at 120.65 125.73)
 		(diameter 0)
@@
 	(wire
 		(pts
+			(xy 209.55 60.96) (xy 209.55 49.53)
+		)
+		(stroke
+			(width 0)
+			(type default)
+		)
+	)
+	(wire
+		(pts
 			(xy 46.99 119.38) (xy 46.99 93.98)
 		)
@@
 	(wire
 		(pts
+			(xy 172.72 63.5) (xy 226.06 63.5)
+		)
+		(stroke
+			(width 0)
+			(type default)
+		)
+	)
+	(wire
+		(pts
 			(xy 115.57 78.74) (xy 151.13 78.74)
 		)
@@
 	(wire
 		(pts
-			(xy 226.06 26.67) (xy 226.06 66.04)
+			(xy 226.06 26.67) (xy 226.06 63.5)
 		)
 		(stroke
@@
 	(wire
 		(pts
+			(xy 228.6 49.53) (xy 228.6 26.67)
+		)
+		(stroke
+			(width 0)
+			(type default)
+		)
+	)
+	(wire
+		(pts
 			(xy 173.99 104.14) (xy 173.99 81.28)
 		)
@@
 	(wire
 		(pts
-			(xy 228.6 62.23) (xy 228.6 26.67)
+			(xy 228.6 62.23) (xy 228.6 49.53)
 		)
 		(stroke
@@
 	(wire
 		(pts
+			(xy 209.55 49.53) (xy 228.6 49.53)
+		)
+		(stroke
+			(width 0)
+			(type default)
+		)
+	)
+	(wire
+		(pts
 			(xy 195.58 113.03) (xy 179.07 113.03)
 		)
@@
 	(wire
 		(pts
+			(xy 172.72 60.96) (xy 209.55 60.96)
+		)
+		(stroke
+			(width 0)
+			(type default)
+		)
+	)
+	(wire
+		(pts
 			(xy 205.74 76.2) (xy 172.72 76.2)
 		)
@@
 		)
 		(stroke
+			(width 0)
+			(type default)
+		)
+	)
+	(wire
+		(pts
+			(xy 226.06 63.5) (xy 226.06 66.04)
+		)
+		(stroke

Commit message: updated pcb files
Parts:
- added J1: GMSB0532112YEU, GMSB0532112YEU:AMPHENOL_GMSB0532112YEU, symbol GMSB0532112YEU:GMSB0532112YEU
- added R14, R15: 22ohm, Resistor_SMD:R_0603_1608Metric_Pad0.98x0.95mm_HandSolder, symbol Device:R
Connections:
- net +5V: now also J1.1 (VBUS)
- net GND: now also J1.5 (GND)
- net at J8.A7 (DN1), J8.B7 (DN2): now also J1.2 (D-), R15.1; no longer U1.26 (GPIO18/USB_D-)
- net at J8.A6 (DP1), J8.B6 (DP2): now also J1.3 (D+), R14.1; no longer U1.27 (GPIO19/USB_D+)
- new net: R15.2, U1.26 (GPIO18/USB_D-)
- new net: J1.S1 (SHIELD), J1.S2 (SHIELD), J1.S3 (SHIELD), J1.S4 (SHIELD)
- new net: R14.2, U1.27 (GPIO19/USB_D+)
Other:
- moved on the sheet: HC-SR501
