File: pcb/Esp32Sensors.kicad_pcb (KiCad board)
At the start: 2 copper layers, 51.8 x 49 mm, 47 parts, among them J8 USB4215-03-A_REVA, U1 ESP32-C3-MINI-1, U10 LM393, U11 LM393, U2 DHT11, U3 DS18B20, U4 AHT20, U5 BMP280, U6 MPU-6050, U7 MAX30102, U8 MCP1702T-3302E_CB, U9 MQ-6

Commit message: updated pcb files
Parts:
- Flame Detector: renamed from D1
- moved C13 2.41 mm to (133.6, 85.2)
- moved C14 2.20 mm to (133.6, 86.8)
- moved C11 1.00 mm to (133.6, 75.8)
- moved C12 1.00 mm to (133.6, 77.4)
- moved U8 1.00 mm to (133.4, 79.6)
- renumbered U4 to AHT20, Feuer-LED to D2, Gas-LED to D3, U2 to DHT11, U3 to DS18B20, U1 to Esp32-C3-Mini-1, R3 to LDR, U7 to MAX30102, U6 to MPU-6050, U9 to MQ-135
Connections:
- Esp32-C3-Mini-1 pad 26: unconnected-(U1-GPIO18/USB_D--Pad26) -> Net-(J8-DN1)
- Esp32-C3-Mini-1 pad 27: unconnected-(U1-GPIO19/USB_D+-Pad27) -> Net-(J8-DP1)
Routing:
- net Net-(J8-DP1): track 2.82 -> 36.7 mm, vias 0 -> 4
- net Net-(J8-DN1): track 2.76 -> 35.4 mm, vias 0 -> 4
- net +5V: track 56.7 -> 50.1 mm
- net GND: track 122.3 -> 115.8 mm, vias 165 -> 170
Other:
- board text added: "BMP280"
- board text added: "IoT Sensors Ref1"

Commit message: updated pcb files
Parts:
- added J1: GMSB0532112YEU, GMSB0532112YEU:AMPHENOL_GMSB0532112YEU, F.Cu at (137.2, 71.8)
- added R14: 22ohm, Resistor_SMD:R_0603_1608Metric_Pad0.98x0.95mm_HandSolder, F.Cu at (115.2, 74.2)
- added R15: 22ohm, Resistor_SMD:R_0603_1608Metric_Pad0.98x0.95mm_HandSolder, F.Cu at (115.2, 75.8)
- D1: renamed from Flame Detector
- moved C12 21.4 mm to (112.4, 80.5), turned to -90 degrees
- moved C11 20.1 mm to (114.0, 80.5), turned to -90 degrees
- moved U8 16.4 mm to (117.0, 80.4), turned to -90 degrees
- moved C13 15.0 mm to (119.8, 79.2), turned to -90 degrees
- moved C14 14.4 mm to (121.4, 79.2), turned to -90 degrees
- moved U7 13.3 mm to (126.6, 68.4)
- renumbered LDR to R3, Esp32-C3-Mini-1 to U1, DHT11 to U2, DS18B20 to U3, AHT20 to U4, MPU-6050 to U6, MAX30102 to U7, MQ-135 to U9
Connections:
- J8 pad A6: Net-(J8-DP1) -> Net-(J1-D+)
- J8 pad A7: Net-(J8-DN1) -> Net-(J1-D-)
- J8 pad B6: Net-(J8-DP1) -> Net-(J1-D+)
- J8 pad B7: Net-(J8-DN1) -> Net-(J1-D-)
- U1 pad 26: Net-(J8-DN1) -> Net-(U1-GPIO18/USB_D-)
- U1 pad 27: Net-(J8-DP1) -> Net-(U1-GPIO19/USB_D+)
Routing:
- net Net-(J1-D+): track 0.00 -> 41.7 mm, vias 0 -> 4
- net Net-(J8-DP1): track 36.7 -> 0.00 mm, vias 4 -> 0
- net Net-(J1-D-): track 0.00 -> 35.9 mm, vias 0 -> 4
- net Net-(J8-DN1): track 35.4 -> 0.00 mm, vias 4 -> 0
- net +5V: track 50.1 -> 71.7 mm, vias 0 -> 2
- net GND: track 115.8 -> 131.5 mm, vias 170 -> 172
- net Net-(U1-GPIO9): track 58.9 -> 50.4 mm, vias 3 -> 2
- net Net-(U1-GPIO19/USB_D+): track 0.00 -> 8.19 mm
- net Net-(U1-GPIO18/USB_D-): track 0.00 -> 8.12 mm
- net Net-(U1-GPIO8): track 57.0 -> 52.6 mm
- net +3.3V: track 173.2 -> 172.3 mm, vias 4 -> 6
Other:
- board text added: "5V"
- board text added: "D0"
- board text added: "GND"

Commit message: updated pcb files
Parts:
- renumbered U3 to DS18B20, D1 to Feuer-LED, D3 to Gas-LED, R2 to LDR, U7 to MAX30102, U6 to MPU-6050, U9 to MQ-135
Routing:
- net +3.3V: track 172.3 -> 182.1 mm, vias 6 -> 8
- net GND: track 131.5 -> 135.8 mm, vias 172 -> 174
